File: Athena.sch (KiCad schematic (older format))
At the start: 79 parts, among them J1 LUM 1503-09, J2 LUM 1503-09, J3 LUM 1503-09, J4 NRJ6HF, J5 DC BU21 90, SW1 MS 500FVT, U1 NE5532, U2 TL072, U3 OPA2134, U4 NE5532, U5 NE5532, U6 NE5532

Commit message: changed enclosure, added power leds, resized pcb
Parts:
- added C13, C14, C15, C16, C17, C18: 100n, Capacitors_SMD:C_0805_HandSoldering, symbol C
- added D2: LED, LEDs:LED_D3.0mm_Horizontal_O3.81mm_Z6.0mm, symbol LED
- added D3: LED, LEDs:LED_D3.0mm_Horizontal_O1.27mm_Z2.0mm, symbol LED
- added J6, J7, J8: NRJ6HF, NRJ6HF:NRJ6HF, symbol Audio-Jack-3_3Switches
- added J9: LUM 1503-09, Lumberg:LUM1503-09, symbol Audio-Jack-3_2Switches
- added R23, R24: 330R, Resistors_SMD:R_0603_HandSoldering, symbol R
- added V31, V32, V33, V34, V35, V36, V37, V38, V39, V40, V41, V42, V43, V44, V45, V46, V47, V48, V49, V50, V51, V52, V53, V54, V55, V56, V57, V58, V59, V60: VIA, via:VIA-0.6, symbol VIA
Connections:
- net +6V: now also C13.1, C15.1, C17.1, R23.1
- net -6V: now also C14.2, C16.2, C18.2, D3.1 (K)
- net GND: now also C13.2, C14.1, C15.2, C16.1, C17.2, C18.1, D2.1 (K), J6.3, J7.3, J8.3, J9.3, R24.1, V31.1, V32.1, V33.1, V34.1, V35.1, V36.1, V37.1, V38.1, V39.1, V40.1, V41.1, V42.1, V43.1, V44.1, V45.1, V46.1, V47.1, V48.1, V49.1, V50.1, V51.1, V52.1, V53.1, V54.1, V55.1, V56.1, V57.1, V58.1, V59.1, V60.1
- net HP_L: now also J9.1
- net HP_R: now also J9.2
- net SUB: now also J8.1
- net TOP_L: now also J7.1
- net TOP_R: now also J7.2
- net at J1.1, RV1.3: now also J6.1
- net at J1.2, RV1.6: now also J6.2
- new net: D2.2 (A), R23.2
- new net: D3.2 (A), R24.2
Other:
- moved on the sheet: C1, C10, C11, C12, C2, C3, C4, C5, C6, C7, C8, C9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
